File: LedChannel.kicad_sch (KiCad schematic)
At the start: 4 parts

Commit message: Schematic: Remove UART channels
Signed-off-by: Geert Uytterhoeven <geert@linux-m68k.org>
Parts:
- renumbered D1 to D2, R1 to R4, R2 to R5, R3 to R6
Changed lines of the file:
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@@
   (symbol (lib_id "Device:R") (at 59.69 38.1 90) (mirror x)
     (in_bom yes) (on_board yes)
-    (property "Reference" "R1" (id 0) (at 58.42 35.56 90)
+    (property "Reference" "R4" (id 0) (at 58.42 35.56 90)
       (effects (font (size 1.27 1.27)) (justify left))
     )
@@
   (symbol (lib_id "Device:R") (at 59.69 43.18 90) (mirror x)
     (in_bom yes) (on_board yes)
-    (property "Reference" "R2" (id 0) (at 58.42 40.64 90)
+    (property "Reference" "R5" (id 0) (at 58.42 40.64 90)
       (effects (font (size 1.27 1.27)) (justify left))
     )
@@
   (symbol (lib_id "Device:R") (at 59.69 48.26 90) (mirror x)
     (in_bom yes) (on_board yes)
-    (property "Reference" "R3" (id 0) (at 58.42 45.72 90)
+    (property "Reference" "R6" (id 0) (at 58.42 45.72 90)
       (effects (font (size 1.27 1.27)) (justify left))
     )
@@
   (symbol (lib_id "Device:LED_ARGB") (at 71.12 43.18 0)
     (in_bom yes) (on_board yes)
-    (property "Reference" "D1" (id 0) (at 71.12 30.5562 0))
+    (property "Reference" "D2" (id 0) (at 71.12 30.5562 0))
     (property "Value" "LED_ARGB" (id 1) (at 71.12 32.8676 0))
     (property "Footprint" "LED_SMD:LED_Cree-PLCC4_3.2x2.8mm_CCW" (id 2) (at 71.12 44.45 0)
