File: OptoChannel.kicad_sch (KiCad schematic)
At the start: 4 parts, among them U6 HCPL-181

Commit message: Schematic: Remove UART channels
Signed-off-by: Geert Uytterhoeven <geert@linux-m68k.org>
Parts:
- renumbered D9 to D10, R25 to R27, R26 to R28, U6 to U7
Changed lines of the file:
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@@
   (symbol (lib_id "Device:R_Small") (at 49.53 35.56 90)
     (in_bom yes) (on_board yes)
-    (property "Reference" "R25" (id 0) (at 49.53 30.48 90))
+    (property "Reference" "R27" (id 0) (at 49.53 30.48 90))
     (property "Value" "1K" (id 1) (at 49.53 33.02 90))
     (property "Footprint" "Resistor_SMD:R_0603_1608Metric_Pad1.05x0.95mm_HandSolder" (id 2) (at 49.53 35.56 0)
@@
   (symbol (lib_id "Device:LED_Small") (at 57.15 35.56 0)
     (in_bom yes) (on_board yes)
-    (property "Reference" "D9" (id 0) (at 57.15 29.591 0))
+    (property "Reference" "D10" (id 0) (at 57.15 29.591 0))
     (property "Value" "Yellow" (id 1) (at 57.15 31.9024 0))
     (property "Footprint" "LED_SMD:LED_0603_1608Metric_Castellated" (id 2) (at 57.15 35.56 90)
@@
   (symbol (lib_id "Device:R_Small") (at 49.53 40.64 90)
     (in_bom yes) (on_board yes)
-    (property "Reference" "R26" (id 0) (at 49.53 43.18 90))
+    (property "Reference" "R28" (id 0) (at 49.53 43.18 90))
     (property "Value" "270" (id 1) (at 49.53 45.72 90))
     (property "Footprint" "Resistor_SMD:R_0603_1608Metric_Pad1.05x0.95mm_HandSolder" (id 2) (at 49.53 40.64 0)
@@
   (symbol (lib_id "Isolator:PC817") (at 72.39 38.1 0)
     (in_bom yes) (on_board yes)
-    (property "Reference" "U6" (id 0) (at 72.39 29.845 0))
+    (property "Reference" "U7" (id 0) (at 72.39 29.845 0))
     (property "Value" "HCPL-181" (id 1) (at 72.39 32.1564 0))
     (property "Footprint" "Package_DIP:SMDIP-4_W7.62mm" (id 2) (at 67.31 43.18 0)

Commit message: Schematic: Re-annotate symbol references
Fill in schematic symbol reference designators, with reset
existing annotations.

Signed-off-by: Geert Uytterhoeven <geert@linux-m68k.org>
Parts:
- renumbered D10 to D8, R27 to R23, R28 to R24, U7 to U9
Changed lines of the file:
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@@
   (symbol (lib_id "Device:R_Small") (at 49.53 35.56 90)
     (in_bom yes) (on_board yes)
-    (property "Reference" "R27" (id 0) (at 49.53 30.48 90))
+    (property "Reference" "R23" (id 0) (at 49.53 30.48 90))
     (property "Value" "1K" (id 1) (at 49.53 33.02 90))
     (property "Footprint" "Resistor_SMD:R_0603_1608Metric_Pad1.05x0.95mm_HandSolder" (id 2) (at 49.53 35.56 0)
@@
   (symbol (lib_id "power:+3V3") (at 62.23 33.02 0)
     (in_bom yes) (on_board yes)
-    (property "Reference" "#PWR018" (id 0) (at 62.23 36.83 0)
+    (property "Reference" "#PWR040" (id 0) (at 62.23 36.83 0)
       (effects (font (size 1.27 1.27)) hide)
     )
@@
   (symbol (lib_id "Device:LED_Small") (at 57.15 35.56 0)
     (in_bom yes) (on_board yes)
-    (property "Reference" "D10" (id 0) (at 57.15 29.591 0))
+    (property "Reference" "D8" (id 0) (at 57.15 29.591 0))
     (property "Value" "Yellow" (id 1) (at 57.15 31.9024 0))
     (property "Footprint" "LED_SMD:LED_0603_1608Metric_Castellated" (id 2) (at 57.15 35.56 90)
@@
   (symbol (lib_id "Device:R_Small") (at 49.53 40.64 90)
     (in_bom yes) (on_board yes)
-    (property "Reference" "R28" (id 0) (at 49.53 43.18 90))
+    (property "Reference" "R24" (id 0) (at 49.53 43.18 90))
     (property "Value" "270" (id 1) (at 49.53 45.72 90))
     (property "Footprint" "Resistor_SMD:R_0603_1608Metric_Pad1.05x0.95mm_HandSolder" (id 2) (at 49.53 40.64 0)
@@
   (symbol (lib_id "Isolator:PC817") (at 72.39 38.1 0)
     (in_bom yes) (on_board yes)
-    (property "Reference" "U7" (id 0) (at 72.39 29.845 0))
+    (property "Reference" "U9" (id 0) (at 72.39 29.845 0))
     (property "Value" "HCPL-181" (id 1) (at 72.39 32.1564 0))
     (property "Footprint" "Package_DIP:SMDIP-4_W7.62mm" (id 2) (at 67.31 43.18 0)

Commit message: Schematic: Update footprints
Update Capacitor, LED, and Resistor footprints to match KiCad 6.

Signed-off-by: Geert Uytterhoeven <geert@linux-m68k.org>
Parts:
- D8: footprint LED_SMD:LED_0603_1608Metric_Castellated -> LED_SMD:LED_0603_1608Metric_Pad1.05x0.95mm_HandSolder
- R23, R24: footprint Resistor_SMD:R_0603_1608Metric_Pad1.05x0.95mm_HandSolder -> Resistor_SMD:R_0603_1608Metric_Pad0.98x0.95mm_HandSolder
Changed lines of the file:
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@@
     (property "Reference" "R23" (id 0) (at 49.53 30.48 90))
     (property "Value" "1K" (id 1) (at 49.53 33.02 90))
-    (property "Footprint" "Resistor_SMD:R_0603_1608Metric_Pad1.05x0.95mm_HandSolder" (id 2) (at 49.53 35.56 0)
+    (property "Footprint" "Resistor_SMD:R_0603_1608Metric_Pad0.98x0.95mm_HandSolder" (id 2) (at 49.53 35.56 0)
       (effects (font (size 1.27 1.27)) hide)
     )
@@
     (property "Reference" "D8" (id 0) (at 57.15 29.591 0))
     (property "Value" "Yellow" (id 1) (at 57.15 31.9024 0))
-    (property "Footprint" "LED_SMD:LED_0603_1608Metric_Castellated" (id 2) (at 57.15 35.56 90)
+    (property "Footprint" "LED_SMD:LED_0603_1608Metric_Pad1.05x0.95mm_HandSolder" (id 2) (at 57.15 35.56 90)
       (effects (font (size 1.27 1.27)) hide)
     )
@@
     (property "Reference" "R24" (id 0) (at 49.53 43.18 90))
     (property "Value" "270" (id 1) (at 49.53 45.72 90))
-    (property "Footprint" "Resistor_SMD:R_0603_1608Metric_Pad1.05x0.95mm_HandSolder" (id 2) (at 49.53 40.64 0)
+    (property "Footprint" "Resistor_SMD:R_0603_1608Metric_Pad0.98x0.95mm_HandSolder" (id 2) (at 49.53 40.64 0)
       (effects (font (size 1.27 1.27)) hide)
     )
