File: BCU-2.kicad_sch (KiCad schematic)
At the start: 14 parts, among them J2 Conn_01x12_Male, J6 Conn_01x04_Male, U1 PCF8574

Commit message: Schematic: Re-annotate symbol references
Fill in schematic symbol reference designators, with reset
existing annotations.

Signed-off-by: Geert Uytterhoeven <geert@linux-m68k.org>
Parts:
- renumbered J2 to J1, J6 to J2, R35 to R1, R36 to R2

Commit message: Schematic: Assign missing footprints
Run footprint assignment tool.

Signed-off-by: Geert Uytterhoeven <geert@linux-m68k.org>
Parts:
- JP1, JP2, JP3, JP4: footprint (none) -> Jumper:SolderJumper-3_P1.3mm_Bridged12_RoundedPad1.0x1.5mm_NumberLabels
- U1: footprint (none) -> Package_SO:SOIC-16W_7.5x10.3mm_P1.27mm
Changed lines of the file:
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@@
       (effects (font (size 1.27 1.27)) (justify left))
     )
-    (property "Footprint" "" (id 2) (at 105.41 137.16 0)
+    (property "Footprint" "Jumper:SolderJumper-3_P1.3mm_Bridged12_RoundedPad1.0x1.5mm_NumberLabels" (id 2) (at 105.41 137.16 0)
       (effects (font (size 1.27 1.27)) hide)
     )
@@
       (effects (font (size 1.27 1.27)) (justify left))
     )
-    (property "Footprint" "" (id 2) (at 54.61 67.31 0)
+    (property "Footprint" "Jumper:SolderJumper-3_P1.3mm_Bridged12_RoundedPad1.0x1.5mm_NumberLabels" (id 2) (at 54.61 67.31 0)
       (effects (font (size 1.27 1.27)) hide)
     )
@@
       (effects (font (size 1.27 1.27)) (justify left))
     )
-    (property "Footprint" "" (id 2) (at 67.31 82.55 0)
+    (property "Footprint" "Jumper:SolderJumper-3_P1.3mm_Bridged12_RoundedPad1.0x1.5mm_NumberLabels" (id 2) (at 67.31 82.55 0)
       (effects (font (size 1.27 1.27)) hide)
     )
@@
       (effects (font (size 1.27 1.27)) (justify left))
     )
-    (property "Footprint" "" (id 2) (at 99.06 69.85 0)
+    (property "Footprint" "Package_SO:SOIC-16W_7.5x10.3mm_P1.27mm" (id 2) (at 99.06 69.85 0)
       (effects (font (size 1.27 1.27)) hide)
     )
@@
       (effects (font (size 1.27 1.27)) (justify left))
     )
-    (property "Footprint" "" (id 2) (at 60.96 74.93 0)
+    (property "Footprint" "Jumper:SolderJumper-3_P1.3mm_Bridged12_RoundedPad1.0x1.5mm_NumberLabels" (id 2) (at 60.96 74.93 0)
       (effects (font (size 1.27 1.27)) hide)
     )
@@
     )
     (path "/2874d169-00ca-4711-b820-9bd76daabb8e"
-      (reference "JP1") (unit 1) (value "SolderJumper_3_Bridged12") (footprint "")
+      (reference "JP1") (unit 1) (value "SolderJumper_3_Bridged12") (footprint "Jumper:SolderJumper-3_P1.3mm_Bridged12_RoundedPad1.0x1.5mm_NumberLabels")
     )
     (path "/f20bea7b-9aea-47e6-889a-0fdfeb98c0ab"
-      (reference "JP2") (unit 1) (value "SolderJumper_3_Bridged12") (footprint "")
+      (reference "JP2") (unit 1) (value "SolderJumper_3_Bridged12") (footprint "Jumper:SolderJumper-3_P1.3mm_Bridged12_RoundedPad1.0x1.5mm_NumberLabels")
     )
     (path "/c61569ba-e093-4c18-ad24-56dd1bfafc07"
-      (reference "JP3") (unit 1) (value "SolderJumper_3_Bridged12") (footprint "")
+      (reference "JP3") (unit 1) (value "SolderJumper_3_Bridged12") (footprint "Jumper:SolderJumper-3_P1.3mm_Bridged12_RoundedPad1.0x1.5mm_NumberLabels")
     )
     (path "/250e396e-532b-403e-9923-ba97292ccd93"
-      (reference "JP4") (unit 1) (value "SolderJumper_3_Bridged12") (footprint "")
+      (reference "JP4") (unit 1) (value "SolderJumper_3_Bridged12") (footprint "Jumper:SolderJumper-3_P1.3mm_Bridged12_RoundedPad1.0x1.5mm_NumberLabels")
     )
     (path "/00000000-0000-0000-0000-00005be8d10d/00000000-0000-0000-0000-00005bf70897"
@@
     )
     (path "/ca56c6fa-1c9a-4c18-af31-0eba468c8eab"
-      (reference "U1") (unit 1) (value "PCF8574") (footprint "")
+      (reference "U1") (unit 1) (value "PCF8574") (footprint "Package_SO:SOIC-16W_7.5x10.3mm_P1.27mm")
     )
     (path "/00000000-0000-0000-0000-00005be8d10d/00000000-0000-0000-0000-00005cf63bde"

Commit message: Schematic: Include DNP I2C pull-up resistors in BOM/board
Else there won't be a footprint in the PCB.

Signed-off-by: Geert Uytterhoeven <geert@linux-m68k.org>
Parts:
- R1, R2: now in the parts list
Changed lines of the file:
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@@
   )
   (symbol (lib_id "Device:R_Small") (at 241.3 95.25 0) (unit 1)
-    (in_bom no) (on_board no)
+    (in_bom yes) (on_board yes)
     (property "Reference" "R1" (id 0) (at 236.22 93.98 0)
       (effects (font (size 1.27 1.27)) (justify left))
@@
   )
   (symbol (lib_id "Device:R_Small") (at 246.38 95.25 0) (unit 1)
-    (in_bom no) (on_board no)
+    (in_bom yes) (on_board yes)
     (property "Reference" "R2" (id 0) (at 247.8786 94.0816 0)
       (effects (font (size 1.27 1.27)) (justify left))

Commit message: Schematic: Update footprints
Update Capacitor, LED, and Resistor footprints to match KiCad 6.

Signed-off-by: Geert Uytterhoeven <geert@linux-m68k.org>
Parts:
- C1: footprint Capacitor_SMD:C_0603_1608Metric_Pad1.05x0.95mm_HandSolder -> Capacitor_SMD:C_0603_1608Metric_Pad1.08x0.95mm_HandSolder
- R1, R2: footprint Resistor_SMD:R_0603_1608Metric_Pad1.05x0.95mm_HandSolder -> Resistor_SMD:R_0603_1608Metric_Pad0.98x0.95mm_HandSolder

Commit message: Schematic: Update title and date
Power-Opto Extension Board (POX for BCU/2)

Signed-off-by: Geert Uytterhoeven <geert@linux-m68k.org>
Other:
- note added: "2023-03-02"
- note added: "Power-Opto Extension Board (POX for BCU/2)"
- note removed: "2019-06-07"
- note removed: "Board Control Unit/2"
Changed lines of the file:
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@@
     (effects (font (size 1.27 1.27)) (justify left bottom))
   )
-  (text "2019-06-07" (at 207.01 194.31 0)
+  (text "2023-03-02" (at 207.01 194.31 0)
     (effects (font (size 1.4986 1.4986)) (justify left bottom))
   )
-  (text "Board Control Unit/2" (at 187.96 190.5 0)
+  (text "Power-Opto Extension Board (POX for BCU/2)" (at 187.96 190.5 0)
     (effects (font (size 1.4986 1.4986)) (justify left bottom))
   )
