File: BCU2-POX.kicad_pcb (KiCad board)
At the start: 2 copper layers, 91.9 x 68 mm, 70 parts, among them J1 Conn_01x12_Male, J2 Conn_01x04_Male, J3 Screw_Terminal_01x04, J4 Screw_Terminal_01x04, Q1 2N7002, Q2 NTF6P02, Q3 2N7002, Q4 2N7002, Q5 NTF6P02, Q6 2N7002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

Commit message: Replace NTF6P02 by DMP6023LE-13
This requires updating the voltage divider providing gate voltage for
the larger Gate Threshold (and Gate-Source) Voltage.

Signed-off-by: Geert Uytterhoeven <geert@linux-m68k.org>
Parts:
- Q2, Q5: value NTF6P02 -> DMP6023LE-13
- R4, R9: value 47K -> 10K
Changed lines of the file:
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@@
       (effects (font (size 1 1) (thickness 0.15)))
     )
-    (fp_text value "47K" (at 0 1.43 90) (layer "F.Fab")
+    (fp_text value "10K" (at 0 1.43 90) (layer "F.Fab")
       (effects (font (size 1 1) (thickness 0.15)))
     )
@@
       (effects (font (size 1 1) (thickness 0.15)))
     )
-    (fp_text value "NTF6P02" (at 3.175 0 180) (layer "F.Fab")
+    (fp_text value "DMP6023LE-13" (at 3.175 0 180) (layer "F.Fab")
       (effects (font (size 1 1) (thickness 0.15)))
     )
@@
       (effects (font (size 1 1) (thickness 0.15)))
     )
-    (fp_text value "47K" (at 0 1.43 -90) (layer "F.Fab")
+    (fp_text value "10K" (at 0 1.43 -90) (layer "F.Fab")
       (effects (font (size 1 1) (thickness 0.15)))
     )
@@
       (effects (font (size 1 1) (thickness 0.15)))
     )
-    (fp_text value "NTF6P02" (at -3.175 0) (layer "F.Fab")
-      (effects (font (size 1 1) (thickness 0.15)))
-    )
+    (fp_text value "DMP6023LE-13" (at -3.175 0) (layer "F.Fab")
+      (effects (font (size 1 1) (thickness 0.15)))
+    )
